File: hardware/InterfaceBoard/SolarHeatingControl.sch (KiCad schematic (older format))
At the start: 39 parts, among them P1 CONN_02X20, P2 CONN_01X02, P3 CONN_01X10, P4 CONN_01X10, U1 CD4051B, U2 OPA2340, U3 OPA2340, U4 MCP3208, U5 CD4051B, U6 MCP23017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

Commit message: add connectors for one-wire-bus and flow-pulse-counter in schematic
Signed-off-by: Christian <christian@dagabumm.ch>
Parts:
- added C12: 1n, symbol C
- added P7: CONN_01X03, symbol CONN_01X03
- added R13: 4K7, symbol R
- added R14: 10K, symbol R
- gave numbers to parts that had none: 8
Connections:
- net labels added: FLOW_PULSE
- wire segments 193 -> 213
Other:
- moved on the sheet: P6
